File: ShieldHardware/IRRxTx.sch (EAGLE design)
At the start: 23 parts, among them IC1 ATMEGA8, J2 Analogs, J4 D8_D13, J5 D0..D7, Q1 16Mhz

Commit message: v.0.07
Added Grenade
Parts:
- added J1: D8_D13, pinhead:PINHD-1X8
- added J3: Analogs, pinhead:PINHD-1X6
- added J6: D0..D7, pinhead:PINHD-1X8
- added JP4: Power_Gnd, SparkFun:M06SIP
Connections:
- new net N$10: JP1.6, JP4.6
- net 3.3V: now also JP4.2
- net AREF: now also J1.8
- net D0: now also J6.1
- net D1: now also J6.2
- net D10: now also J1.3
- net D11: now also J1.4
- net D12: now also J1.5
- net D13: now also J1.6
- net D18: now also J3.5
- net D2: now also J6.3
- net D3: now also J6.4
- net D4: now also J6.5
- net D5: now also J6.6
- net D6: now also J6.7
- net D7: now also J6.8
- net D8: now also J1.1
- net D9: now also J1.2
- net GND: now also J1.7, JP4.4, JP4.5
- net N$16: now also J3.1
- net N$17: now also J3.2
- net N$18: now also J3.3
- net N$19: now also J3.4
- net N$21: now also J3.6
- net RST: now also JP4.1
- net VCC: now also JP4.3
Changed lines of the file:
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@@
 <setting verticaltext="up"/>
 </settings>
-<grid distance="0.05" unitdist="inch" unit="inch" style="lines" multiple="1" display="no" altdistance="0.01" altunitdist="inch" altunit="inch"/>
+<grid distance="0.1" unitdist="inch" unit="inch" style="lines" multiple="1" display="no" altdistance="0.01" altunitdist="inch" altunit="inch"/>
 <layers>
 <layer number="1" name="Top" color="4" fill="1" visible="no" active="no"/>
@@
 <part name="GND13" library="SparkFun" deviceset="GND" device=""/>
 <part name="P+5" library="SparkFun" deviceset="VCC" device=""/>
+<part name="J1" library="pinhead" deviceset="PINHD-1X8" device="" value="D8_D13"/>
+<part name="J3" library="pinhead" deviceset="PINHD-1X6" device="" value="Analogs"/>
+<part name="J6" library="pinhead" deviceset="PINHD-1X8" device="" value="D0..D7"/>
+<part name="JP4" library="SparkFun" deviceset="M06" device="SIP" value="Power_Gnd"/>
 </parts>
 <sheets>
@@
 <instance part="GND13" gate="1" x="-2.54" y="30.48"/>
 <instance part="P+5" gate="1" x="-15.24" y="45.72" rot="R90"/>
+<instance part="J1" gate="A" x="241.3" y="83.82" rot="MR180"/>
+<instance part="J3" gate="A" x="212.09" y="58.42" rot="MR180"/>
+<instance part="J6" gate="A" x="228.6" y="33.02" rot="MR180"/>
+<instance part="JP4" gate="G$1" x="100.33" y="111.76" rot="R180"/>
 </instances>
 <busses>
@@
 <label x="196.215" y="88.9" size="1.778" layer="95"/>
 <pinref part="J4" gate="A" pin="7"/>
+<pinref part="J1" gate="A" pin="7"/>
+<junction x="238.76" y="88.9"/>
 </segment>
 <segment>
@@
 <pinref part="GND10" gate="1" pin="GND"/>
 <pinref part="JP1" gate="G$1" pin="4"/>
+<pinref part="JP4" gate="G$1" pin="4"/>
+<junction x="95.25" y="109.22"/>
+<pinref part="JP4" gate="G$1" pin="5"/>
+<junction x="95.25" y="106.68"/>
 </segment>
 <segment>
@@
 <pinref part="IC1" gate="G$1" pin="(ADC0)PC0)"/>
 <pinref part="J2" gate="A" pin="1"/>
+<pinref part="J3" gate="A" pin="1"/>
+<junction x="209.55" y="50.8"/>
 </segment>
 </net>
@@
 <pinref part="IC1" gate="G$1" pin="(ADC1)PC1"/>
 <pinref part="J2" gate="A" pin="2"/>
+<pinref part="J3" gate="A" pin="2"/>
+<junction x="209.55" y="53.34"/>
 </segment>
 </net>
@@
 <pinref part="IC1" gate="G$1" pin="(ADC2)PC2"/>
 <pinref part="J2" gate="A" pin="3"/>
+<pinref part="J3" gate="A" pin="3"/>
+<junction x="209.55" y="55.88"/>
 </segment>
 </net>
@@
 <pinref part="IC1" gate="G$1" pin="(ADC3)PC3"/>
 <pinref part="J2" gate="A" pin="4"/>
+<pinref part="J3" gate="A" pin="4"/>
+<junction x="209.55" y="58.42"/>
 </segment>
 </net>
@@
 <pinref part="IC1" gate="G$1" pin="(ADC5)PC5"/>
 <pinref part="J2" gate="A" pin="6"/>
+<pinref part="J3" gate="A" pin="6"/>
+<junction x="209.55" y="63.5"/>
 </segment>
 </net>
@@
 <label x="196.215" y="92.075" size="1.778" layer="95"/>
 <pinref part="J4" gate="A" pin="8"/>
+<pinref part="J1" gate="A" pin="8"/>
+<junction x="238.76" y="91.44"/>
 </segment>
 </net>
@@
 <pinref part="JP1" gate="G$1" pin="3"/>
 <pinref part="P+6" gate="1" pin="VCC"/>
+<pinref part="JP4" gate="G$1" pin="3"/>
+<junction x="95.25" y="111.76"/>
 </segment>
 <segment>
@@
 <label x="207.01" y="73.66" size="1.778" layer="95"/>
 <pinref part="J4" gate="A" pin="1"/>
+<pinref part="J1" gate="A" pin="1"/>
+<junction x="238.76" y="73.66"/>
 </segment>
 <segment>
@@
 <label x="207.01" y="78.74" size="1.778" layer="95"/>
 <pinref part="J4" gate="A" pin="3"/>
+<pinref part="J1" gate="A" pin="3"/>
+<junction x="238.76" y="78.74"/>
 </segment>
 <segment>
@@
 <label x="201.93" y="76.2" size="1.778" layer="95"/>
 <pinref part="J4" gate="A" pin="2"/>
+<pinref part="J1" gate="A" pin="2"/>
+<junction x="238.76" y="76.2"/>
 </segment>
 <segment>
@@
 <label x="201.93" y="81.28" size="1.778" layer="95"/>
 <pinref part="J4" gate="A" pin="4"/>
+<pinref part="J1" gate="A" pin="4"/>
+<junction x="238.76" y="81.28"/>
 </segment>
 <segment>
@@
 <label x="207.01" y="83.82" size="1.778" layer="95"/>
 <pinref part="J4" gate="A" pin="5"/>
+<pinref part="J1" gate="A" pin="5"/>
+<junction x="238.76" y="83.82"/>
 </segment>
 <segment>
@@
 <label x="201.93" y="86.36" size="1.778" layer="95"/>
 <pinref part="J4" gate="A" pin="6"/>
+<pinref part="J1" gate="A" pin="6"/>
+<junction x="238.76" y="86.36"/>
 </segment>
 </net>
@@
 <label x="200.66" y="60.96" size="1.778" layer="95"/>
 <pinref part="J2" gate="A" pin="5"/>
+<pinref part="J3" gate="A" pin="5"/>
+<junction x="209.55" y="60.96"/>
 </segment>
 </net>
@@
 <label x="232.41" y="22.86" size="1.778" layer="95"/>
 <pinref part="J5" gate="A" pin="1"/>
+<pinref part="J6" gate="A" pin="1"/>
+<junction x="226.06" y="22.86"/>
 </segment>
 <segment>
@@
 <label x="232.41" y="25.4" size="1.778" layer="95"/>
 <pinref part="J5" gate="A" pin="2"/>
+<pinref part="J6" gate="A" pin="2"/>
+<junction x="226.06" y="25.4"/>
 </segment>
 <segment>
@@
 <label x="87.63" y="114.3" size="1.778" layer="95"/>
 <pinref part="JP1" gate="G$1" pin="2"/>
+<pinref part="JP4" gate="G$1" pin="2"/>
+<junction x="95.25" y="114.3"/>
 </segment>
 <segment>
@@
 <label x="212.09" y="35.56" size="1.778" layer="95"/>
 <pinref part="J5" gate="A" pin="6"/>
+<pinref part="J6" gate="A" pin="6"/>
+<junction x="226.06" y="35.56"/>
 </segment>
 </net>
@@
 <label x="218.44" y="38.1" size="1.778" layer="95"/>
 <pinref part="J5" gate="A" pin="7"/>
+<pinref part="J6" gate="A" pin="7"/>
+<junction x="226.06" y="38.1"/>
 </segment>
 </net>
@@
 <label x="212.09" y="40.64" size="1.778" layer="95"/>
 <pinref part="J5" gate="A" pin="8"/>
+<pinref part="J6" gate="A" pin="8"/>
+<junction x="226.06" y="40.64"/>
 </segment>
 </net>
@@
 <label x="212.09" y="27.94" size="1.778" layer="95"/>
 <pinref part="J5" gate="A" pin="3"/>
+<pinref part="J6" gate="A" pin="3"/>
+<junction x="226.06" y="27.94"/>
 </segment>
 </net>
@@
 <label x="217.17" y="30.48" size="1.778" layer="95"/>
 <pinref part="J5" gate="A" pin="4"/>
+<pinref part="J6" gate="A" pin="4"/>
+<junction x="226.06" y="30.48"/>
 </segment>
 <segment>
@@
 <label x="212.09" y="33.02" size="1.778" layer="95"/>
 <pinref part="J5" gate="A" pin="5"/>
+<pinref part="J6" gate="A" pin="5"/>
+<junction x="226.06" y="33.02"/>
 </segment>
 </net>
@@
 <label x="76.2" y="116.84" size="1.778" layer="95"/>
 <pinref part="JP1" gate="G$1" pin="1"/>
+<pinref part="JP4" gate="G$1" pin="1"/>
+<junction x="95.25" y="116.84"/>
 </segment>
 </net>
@@
 </segment>
 </net>
+<net name="N$10" class="0">
+<segment>
+<pinref part="JP1" gate="G$1" pin="6"/>
+<pinref part="JP4" gate="G$1" pin="6"/>
+</segment>
+</net>
